Commit message: fixed car's orientation

File: urdf/car.urdf.xacro (robot description, xacro)
@@ -169,5 +169,5 @@
     <parent link="lidar_link"/>
     <child link="lidar_scan_frame"/>
-    <origin xyz="0 0 0" rpy="0 0 0"/>
+    <origin xyz="0 0 0" rpy="0 0 3.14159265359"/>
   </joint>
   <ros2_control name="ackermann_mock_system" type="system">
